File: Kicad/Neotron-9X-CPU/Neotron-9X-CPU.kicad_pcb (KiCad board)
At the start: 2 copper layers, 170 x 170 mm, 5 parts, among them U101 SAM9X60D5M

Commit message: Split into separate mainboard and CPU board projects.
Parts:
- U101: footprint Neotron-9X:BGA-233_17x17_14.0x14.0mm -> Neotron-9X-CPU:BGA-233_17x17_14.0x14.0mm
Changed lines of the file:
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@@
     )
   )
-  (module Neotron-9X:BGA-233_17x17_14.0x14.0mm (layer F.Cu)
+  (module Neotron-9X-CPU:BGA-233_17x17_14.0x14.0mm (layer F.Cu)
     (at 140 145)
     (attr smd)
