File: Kicad/Neotron-9X-CPU/Neotron-9X-CPU.sch (KiCad schematic (older format))
At the start: 38 parts, among them J1 JTAG Header, U1 SAM9X60D5M

Commit message: Starting on VGA DAC.
Parts:
- gave numbers to parts that had none: 1
Connections:
- net labels added: HHSDA+, HHSDA-, IO_POWER
- net labels removed: USBA+, USBA-
- wire segments 533 -> 546
Other:
- note removed: "Super VGA DAC"
- moved on the sheet: U101
