File: Kicad/Neotron-Base/rtc.sch (KiCad schematic (older format))
At the start: 6 parts, among them U301 MCP7940N-xP, Y301 32,768 Hz

Commit message: Re-work CPU interface to include RMII.
Parts:
- renumbered C303 to C302, C302 to C303
Changed lines of the file:
@@
 $Descr A4 11693 8268
 encoding utf-8
-Sheet 3 7
+Sheet 3 10
 Title "Neotron Base - Real Time Clock"
-Date "2020-08-07"
+Date "2020-08-15"
 Rev "[Uncontrolled]"
 Comp "github.com/neotron-compute"
@@
 AR Path="/5DF1D0B0/5E0203CB" Ref="C?"  Part="1"
 AR Path="/5DF66898/5E0203CB" Ref="C?"  Part="1"
-AR Path="/5F3C1328/5E0203CB" Ref="C302"  Part="1"
-F 0 "C302" H 7165 3396 50  0000 L CNN
+AR Path="/5F3C1328/5E0203CB" Ref="C303"  Part="1"
+F 0 "C303" H 7165 3396 50  0000 L CNN
 F 1 "100n" H 7165 3305 50  0000 L CNN
 F 2 "Capacitor_THT:C_Disc_D3.0mm_W2.0mm_P2.50mm" H 7088 3200 50  0001 C CNN
@@
 $EndComp
 $Comp
-L Device:C C303
+L Device:C C302
 U 1 1 5E02CC31
 P 5550 3750
-F 0 "C303" H 5665 3796 50  0000 L CNN
+F 0 "C302" H 5665 3796 50  0000 L CNN
 F 1 "6p" H 5665 3705 50  0000 L CNN
 F 2 "Capacitor_THT:C_Disc_D3.0mm_W2.0mm_P2.50mm" H 5588 3600 50  0001 C CNN
